File: BCU-2.kicad_pcb (KiCad board)
At the start: 2 copper layers, 106 x 91.4 mm, 92 parts, among them J1 Screw_Terminal_01x04, J2 Conn_01x12_Male, J3 Screw_Terminal_01x04, J4 Conn_01x05_Male, J5 Conn_01x05_Male, J6 Conn_01x04_Male, J7 Conn_01x04_Male, Q1 2N7002, Q2 NTF6P02, Q3 2N7002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

Commit message: Improve silkscreen for rev1.01
Signed-off-by: Geert Uytterhoeven <geert@linux-m68k.org>
Other:
- board text added: "+3V3"
- board text added: "- +"
- board text added: "BCU/2 rev1.01"
- board text added: "Channel A"
- board text added: "Channel B"
- board text added: "GND"
- board text added: "GPIO0"
- board text added: "GPIO1"
- board text added: "IN"
- board text added: "OUT"
- board text added: "P0"
- board text added: "P1"
- board text added: "P2"
- board text added: "P3"
- board text added: "P4"
- board text added: "P5"
- board text added: "RXD"
- board text added: "SCL"
- board text added: "SDA"
- board text added: "TXD"
- board text added: "VBUS"
- board text removed: "BCU/2 rev1.0"
Changed lines of the file:
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@@
-(kicad_pcb (version 20171130) (host pcbnew 5.0.2-bee76a0~70~ubuntu18.04.1)
+(kicad_pcb (version 20171130) (host pcbnew 5.1.5+dfsg1-2build2)
   (general
     (thickness 1.6)
-    (drawings 9)
+    (drawings 49)
     (tracks 443)
     (zones 0)
@@
     (zone_45_only no)
     (trace_min 0.2)
-    (segment_width 0.2)
-    (edge_width 0.15)
     (via_size 0.8)
     (via_drill 0.4)
@@
     (uvia_min_size 0.2)
     (uvia_min_drill 0.1)
+    (edge_width 0.15)
+    (segment_width 0.2)
     (pcb_text_width 0.3)
     (pcb_text_size 1.5 1.5)
@@
     (pad 20 thru_hole circle (at 16.51 -7.62 270) (size 1.6 1.6) (drill 1.1) (layers *.Cu *.Mask F.SilkS))
   )
+  (gr_text "Channel A" (at 115.824 96.52) (layer F.SilkS)
+    (effects (font (size 2 2) (thickness 0.4)))
+  )
+  (gr_text "Channel B" (at 201.93 74.93) (layer F.SilkS)
+    (effects (font (size 2 2) (thickness 0.4)))
+  )
+  (gr_text P5 (at 171.45 132.08) (layer F.SilkS)
+    (effects (font (size 1.1 1.1) (thickness 0.15)))
+  )
+  (gr_text P4 (at 166.37 132.08) (layer F.SilkS)
+    (effects (font (size 1.1 1.1) (thickness 0.15)))
+  )
+  (gr_text P3 (at 161.29 132.08) (layer F.SilkS)
+    (effects (font (size 1.1 1.1) (thickness 0.15)))
+  )
+  (gr_text P2 (at 156.21 132.08) (layer F.SilkS)
+    (effects (font (size 1.1 1.1) (thickness 0.15)))
+  )
+  (gr_text "- +" (at 171.45 130.937) (layer F.SilkS)
+    (effects (font (size 1.1 1.25) (thickness 0.15)))
+  )
+  (gr_text "- +" (at 166.37 130.937) (layer F.SilkS)
+    (effects (font (size 1.1 1.25) (thickness 0.15)))
+  )
+  (gr_text "- +" (at 161.29 130.937) (layer F.SilkS)
+    (effects (font (size 1.1 1.25) (thickness 0.15)))
+  )
+  (gr_text "- +" (at 156.21 130.937) (layer F.SilkS)
+    (effects (font (size 1.1 1.25) (thickness 0.15)))
+  )
+  (gr_text "- +" (at 151.13 130.937) (layer F.SilkS)
+    (effects (font (size 1.1 1.25) (thickness 0.15)))
+  )
+  (gr_text P1 (at 151.13 132.08) (layer F.SilkS)
+    (effects (font (size 1.1 1.1) (thickness 0.15)))
+  )
+  (gr_text "- +" (at 146.05 130.937) (layer F.SilkS)
+    (effects (font (size 1.1 1.25) (thickness 0.15)))
+  )
+  (gr_text P0 (at 146.05 132.08) (layer F.SilkS)
+    (effects (font (size 1.1 1.1) (thickness 0.15)))
+  )
+  (gr_text GPIO1 (at 141.732 51.816 90) (layer F.SilkS)
+    (effects (font (size 1.2 1.2) (thickness 0.2)) (justify right))
+  )
+  (gr_text GPIO0 (at 139.7 51.816 90) (layer F.SilkS)
+    (effects (font (size 1.2 1.2) (thickness 0.2)) (justify right))
+  )
+  (gr_text +3V3 (at 137.668 51.816 90) (layer F.SilkS)
+    (effects (font (size 1.2 1.2) (thickness 0.2)) (justify right))
+  )
+  (gr_text GND (at 135.636 51.816 90) (layer F.SilkS)
+    (effects (font (size 1.2 1.2) (thickness 0.2)) (justify right))
+  )
+  (gr_text SCL (at 183.388 51.816 90) (layer F.SilkS)
+    (effects (font (size 1.2 1.2) (thickness 0.2)) (justify right))
+  )
+  (gr_text SDA (at 181.356 51.816 90) (layer F.SilkS)
+    (effects (font (size 1.2 1.2) (thickness 0.2)) (justify right))
+  )
+  (gr_text +3V3 (at 179.324 51.816 90) (layer F.SilkS)
+    (effects (font (size 1.2 1.2) (thickness 0.2)) (justify right))
+  )
+  (gr_text GND (at 177.292 51.816 90) (layer F.SilkS)
+    (effects (font (size 1.2 1.2) (thickness 0.2)) (justify right))
+  )
+  (gr_text +3V3 (at 114.681 68.199) (layer F.SilkS)
+    (effects (font (size 1.4 1.4) (thickness 0.25)) (justify right))
+  )
+  (gr_text VBUS (at 114.681 65.659) (layer F.SilkS)
+    (effects (font (size 1.4 1.4) (thickness 0.25)) (justify right))
+  )
+  (gr_text TXD (at 114.681 63.119) (layer F.SilkS)
+    (effects (font (size 1.4 1.4) (thickness 0.25)) (justify right))
+  )
+  (gr_text RXD (at 114.681 60.579) (layer F.SilkS)
+    (effects (font (size 1.4 1.4) (thickness 0.25)) (justify right))
+  )
+  (gr_text GND (at 114.681 58.039) (layer F.SilkS)
+    (effects (font (size 1.4 1.4) (thickness 0.25)) (justify right))
+  )
+  (gr_text +3V3 (at 202.438 57.912) (layer F.SilkS)
+    (effects (font (size 1.4 1.4) (thickness 0.25)) (justify left))
+  )
+  (gr_text VBUS (at 202.946 60.452) (layer F.SilkS)
+    (effects (font (size 1.4 1.4) (thickness 0.25)) (justify left))
+  )
+  (gr_text TXD (at 202.946 62.992) (layer F.SilkS)
+    (effects (font (size 1.4 1.4) (thickness 0.25)) (justify left))
+  )
+  (gr_text RXD (at 202.946 65.532) (layer F.SilkS)
+    (effects (font (size 1.4 1.4) (thickness 0.25)) (justify left))
+  )
+  (gr_text GND (at 202.946 68.072) (layer F.SilkS)
+    (effects (font (size 1.4 1.4) (thickness 0.25)) (justify left))
+  )
+  (gr_text OUT (at 206.248 92.456) (layer F.SilkS)
+    (effects (font (size 1.5 1.5) (thickness 0.3)) (justify left))
+  )
+  (gr_text IN (at 206.248 85.344) (layer F.SilkS)
+    (effects (font (size 1.5 1.5) (thickness 0.3)) (justify left))
+  )
+  (gr_text GND (at 206.248 96.012) (layer F.SilkS)
+    (effects (font (size 1.5 1.5) (thickness 0.3)) (justify left))
+  )
+  (gr_text GND (at 206.248 88.9) (layer F.SilkS)
+    (effects (font (size 1.5 1.5) (thickness 0.3)) (justify left))
+  )
+  (gr_text "IN\n" (at 111.252 87.376) (layer F.SilkS)
+    (effects (font (size 1.5 1.5) (thickness 0.3)) (justify right))
+  )
+  (gr_text GND (at 111.252 83.82) (layer F.SilkS)
+    (effects (font (size 1.5 1.5) (thickness 0.3)) (justify right))
+  )
+  (gr_text "OUT\n" (at 111.252 80.264) (layer F.SilkS)
+    (effects (font (size 1.5 1.5) (thickness 0.3)) (justify right))
+  )
+  (gr_text GND (at 111.252 76.835) (layer F.SilkS)
+    (effects (font (size 1.5 1.5) (thickness 0.3)) (justify right))
+  )
   (gr_line (start 111.125 133.985) (end 207.01 133.985) (layer Edge.Cuts) (width 0.15))
   (gr_line (start 106.045 47.625) (end 106.045 128.905) (layer Edge.Cuts) (width 0.15))
@@
   (gr_arc (start 207.01 47.625) (end 212.09 47.625) (angle -90) (layer Edge.Cuts) (width 0.15))
   (gr_arc (start 111.125 47.625) (end 111.125 42.545) (angle -90) (layer Edge.Cuts) (width 0.15))
-  (gr_text "BCU/2 rev1.0\n" (at 196.215 119.38) (layer F.SilkS)
+  (gr_text "BCU/2 rev1.01" (at 196.215 119.38) (layer F.SilkS)
     (effects (font (size 1.5 1.5) (thickness 0.3)))
   )
